File: _autosave-Urban MC.kicad_sch (KiCad schematic)
At the start: 47 parts, among them J1 Conn_01x02, J2 Screw_Terminal_01x02, J3 Conn_01x02, J4 Conn_01x03, J5 Conn_01x02, SW1 SW_Push, U1 IRS2186, U1 MCP4725xxx-xCH, U2 IRS2186, U2 MCP2515-xSO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

Commit message: error fixes
Parts:
- added J6: Screw_Terminal_01x03, symbol Connector:Screw_Terminal_01x03
Connections:
- net VCC is gone; now on an unnamed net: U3.3 (VCC)
- net +48V: now also J6.1 (Pin_1), J6.2 (Pin_2), J6.3 (Pin_3)
Other:
- moved on the sheet: A1, C1, C10, C11, C12, C13, C2, C3, C4, C5, C6, C7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
