File: Urban MC.kicad_pcb (KiCad board)
At the start: 4 copper layers, 167 x 104 mm, 72 parts, among them J1 Conn_01x02, J2 Conn_01x02, J3 Screw_Terminal_01x02, J4 Screw_Terminal_01x01, J5 Screw_Terminal_01x01, J6 Screw_Terminal_01x01, J7 Screw_Terminal_01x01, J8 Screw_Terminal_01x01, Q1 IQE022N06LM5CGSCATMA1, Q10 IQE022N06LM5CGSCATMA1, Q11 IQE022N06LM5CGSCATMA1, Q12 IQE022N06LM5CGSCATMA1, Q13 IQE022N06LM5CGSCATMA1, Q14 IQE022N06LM5CGSCATMA1, Q15 IQE022N06LM5CGSCATMA1, Q16 IQE022N06LM5CGSCATMA1, Q17 IQE022N06LM5CGSCATMA1, Q18 IQE022N06LM5CGSCATMA1, Q19 IQE022N06LM5CGSCATMA1, Q2 IQE022N06LM5CGSCATMA1, Q20 IQE022N06LM5CGSCATMA1, Q21 IQE022N06LM5CGSCATMA1, Q22 IQE022N06LM5CGSCATMA1, Q23 IQE022N06LM5CGSCATMA1, Q24 IQE022N06LM5CGSCATMA1, Q3 IQE022N06LM5CGSCATMA1, Q4 IQE022N06LM5CGSCATMA1, Q5 IQE022N06LM5CGSCATMA1, Q6 IQE022N06LM5CGSCATMA1, Q7 IQE022N06LM5CGSCATMA1, Q8 IQE022N06LM5CGSCATMA1, Q9 IQE022N06LM5CGSCATMA1, SW1 SW_Push, U1 IRS2186, U11 MCP2515-xSO, U12 TJA1050, U13 MCP4725, U2 IRS2186, U3 IRS2186

Commit message: mosfets
Parts:
- moved C5 54.8 mm to (167.3, 78.7), turned to 90 degrees
- moved R3 54.5 mm to (168.5, 85.1)
- moved C8 45.8 mm to (167.6, 102.5), turned to 90 degrees
- moved C4 43.6 mm to (161.0, 85.7)
- moved R7 42.6 mm to (167.4, 106.7)
- moved R2 37.9 mm to (172.6, 73.0)
- moved C7 36.5 mm to (160.3, 107.0)
- moved R4 35.4 mm to (166.9, 73.7)
- moved R10 34.0 mm to (162.8, 134.0)
- moved C11 33.6 mm to (157.2, 135.3), turned to 180 degrees
- moved C10 32.8 mm to (157.8, 120.0), turned to 180 degrees
- moved R9 30.8 mm to (168.2, 133.3)
- moved Q19 30.7 mm to (184.8, 127.6)
- moved Q17 30.3 mm to (170.2, 127.6)
- moved Q1 29.4 mm to (173.7, 79.5), turned to 90 degrees
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- renumbered Q11 to Q10, Q13 to Q11, Q15 to Q12, Q10 to Q13, Q12 to Q14, Q14 to Q15, Q19 to Q18, Q21 to Q19, Q23 to Q20, Q18 to Q21, Q20 to Q22, Q22 to Q23

Commit message: MOSFET section draft
Parts:
- moved R4 35.8 mm to (200.2, 87.0)
- moved D2 10.2 mm to (161.3, 69.8), turned to 180 degrees
- moved R3 3.19 mm to (168.7, 81.9)
- moved C4 2.84 mm to (162.2, 83.2)
- moved R2 1.63 mm to (171.6, 71.8)
- moved C6 1.42 mm to (205.1, 80.6), turned to 90 degrees
- moved Q8 1.15 mm to (235.2, 79.4), turned to 90 degrees
- moved C5 1.07 mm to (166.4, 78.1)
- moved Q7 1.01 mm to (228.7, 79.3), turned to 90 degrees
- moved Q5 0.75 mm to (213.9, 79.5), turned to 90 degrees
- moved Q6 0.51 mm to (221.4, 79.4), turned to 90 degrees
- moved Q4 0.08 mm to (196.1, 79.5), turned to -90 degrees
- turned Q1 to -90 degrees
- turned Q2 to -90 degrees
- turned Q3 to -90 degrees
Routing:
- net Net-(Q5-GATE): track 0.00 -> 72.2 mm, vias 0 -> 5
- net Net-(Q1-GATE): track 0.00 -> 66.6 mm, vias 0 -> 5
- net Net-(U1-LO): track 0.00 -> 45.4 mm
- net +12V: track 0.00 -> 21.1 mm
- net Net-(U1-HO): track 0.00 -> 14.4 mm
- net Net-(D2-K): track 0.00 -> 12.0 mm, vias 0 -> 2
- net Net-(U1-VS): track 0.00 -> 6.75 mm
- net Net-(J8-Pin_1): track 0.00 -> 6.15 mm
- net GND: track 0.00 -> 5.41 mm
- added copper zone on F.Cu, net +48V
- added copper zone on B.Cu, net GND
- added copper zone on F.Cu, net Net-(J8-Pin_1)

Commit message: MOSFETsection with some changes
Parts:
- removed the C12 at (203.0, 127.9)
- removed the C6 at (205.1, 80.6)
- removed the C8 at (167.6, 102.5)
- removed the D4 at (152.4, 132.1)
- removed J6, J7, J8: Screw_Terminal_01x01, urban_mc_custom_footprints:WP-SHFU_7461100
- removed the Q13 at (214.0, 102.2)
- removed the Q14 at (221.6, 101.6)
- removed the Q15 at (229.2, 101.6)
- removed the Q16 at (236.3, 102.0)
- removed the Q17 at (170.2, 127.6)
- removed the Q18 at (177.2, 127.6)
- removed the Q19 at (184.8, 127.6)
- removed the Q20 at (192.0, 127.8)
- removed the R11 at (23.8, 152.5)
- removed the R6 at (172.6, 96.5)
- removed the R7 at (167.4, 106.7)
- removed the U2 at (160.7, 101.0)
- added C1: 10u, Capacitor_SMD:C_0805_2012Metric, F.Cu at (139.3, 61.5)
- added C10: 1u, Capacitor_SMD:C_2220_5750Metric, F.Cu at (203.2, 71.1)
- added C2: 0.1uF, Capacitor_SMD:C_0805_2012Metric_Pad1.18x1.45mm_HandSolder, F.Cu at (139.5, 70.5)
- added C3: 10u, Capacitor_SMD:C_0805_2012Metric, F.Cu at (139.7, 64.5)
- added C4: 10u, Capacitor_SMD:C_0805_2012Metric, F.Cu at (139.7, 67.3)
- added C5: 1u, Capacitor_SMD:C_2220_5750Metric, F.Cu at (124.5, 99.1)
- added D1: D, urban_mc_custom_footprints:DIODE_DO214AA_MBRS_VIS, F.Cu at (123.2, 72.4)
- added G1: IRS2186, Package_SO:SOIC-8_3.9x4.9mm_P1.27mm, F.Cu at (132.8, 63.4)
- added J2: Conn_01x02, urban_mc_custom_footprints:CON_436500200_MOL, F.Cu at (137.7, 82.9)
- added J3: Conn_01x03, urban_mc_custom_footprints:TE_1986660-3, F.Cu at (257.8, 93.0)
- added J4: Conn_01x02, urban_mc_custom_footprints:TE_1-1986660-2, F.Cu at (102.4, 93.8)
- added Q1: IQE022N06LM5CGSCATMA1, urban_mc_custom_footprints:IFX-PG-WHTFN-9-1-V, F.Cu at (99.2, 82.8)
- added Q2: IQE022N06LM5CGSCATMA1, urban_mc_custom_footprints:IFX-PG-WHTFN-9-1-V, F.Cu at (99.2, 88.5)
- added Q3: IQE022N06LM5CGSCATMA1, urban_mc_custom_footprints:IFX-PG-WHTFN-9-1-V, F.Cu at (105.3, 82.8)
- added Q4: IQE022N06LM5CGSCATMA1, urban_mc_custom_footprints:IFX-PG-WHTFN-9-1-V, F.Cu at (105.3, 88.5)
- added Q5: IQE022N06LM5CGSCATMA1, urban_mc_custom_footprints:IFX-PG-WHTFN-9-1-V, F.Cu at (111.5, 82.8)
- added Q6: IQE022N06LM5CGSCATMA1, urban_mc_custom_footprints:IFX-PG-WHTFN-9-1-V, F.Cu at (111.5, 88.5)
- added Q7: IQE022N06LM5CGSCATMA1, urban_mc_custom_footprints:IFX-PG-WHTFN-9-1-V, F.Cu at (117.6, 82.8)
- added Q8: IQE022N06LM5CGSCATMA1, urban_mc_custom_footprints:IFX-PG-WHTFN-9-1-V, F.Cu at (117.6, 88.5)
- added R1: 120, Resistor_SMD:R_0603_1608Metric, F.Cu at (130.6, 74.4)
- added R2: 11Ω, Resistor_SMD:R_0402_1005Metric, F.Cu at (135.7, 108.5)
- added R3: 2.4Ω, Resistor_SMD:R_0603_1608Metric, F.Cu at (130.6, 76.9)
- added R4: 10k, Resistor_SMD:R_0805_2012Metric_Pad1.20x1.40mm_HandSolder, F.Cu at (123.2, 110.5)
- added SW1: CAN_TERM, Connector_PinHeader_2.54mm:PinHeader_1x02_P2.54mm_Horizontal, F.Cu at (131.8, 95.9)
- added U1: MCP2561/2, Package_SO:SOIC-8_3.9x4.9mm_P1.27mm, F.Cu at (132.8, 69.9)
- added Y1: 8MHz, Crystal:Crystal_HC49-U_Vertical, F.Cu at (133.6, 104.1)
- C13: value 10u -> 1u; footprint Capacitor_SMD:C_0805_2012Metric -> Capacitor_SMD:C_2220_5750Metric
- C7: value 10u -> 16pF; footprint Capacitor_SMD:C_0805_2012Metric -> Capacitor_SMD:C_0805_2012Metric_Pad1.18x1.45mm_HandSolder
- C9: value 1u -> 16pF; footprint Capacitor_SMD:C_2220_5750Metric -> Capacitor_SMD:C_0805_2012Metric_Pad1.18x1.45mm_HandSolder
- D2, D3: footprint Diode_THT:D_DO-41_SOD81_P10.16mm_Horizontal -> urban_mc_custom_footprints:DIODE_DO214AA_MBRS_VIS
- D4: renamed from D1; footprint Diode_THT:D_DO-41_SOD81_P10.16mm_Horizontal -> urban_mc_custom_footprints:DO-201AD
- moved C13 183.6 mm to (201.9, 125.1), turned to 90 degrees
- moved C9 69.7 mm to (139.5, 76.6)
- moved R9 58.9 mm to (166.8, 62.4)
- moved R8 57.0 mm to (163.2, 77.0)
- moved C6 57.0 mm to (158.2, 63.0)
- moved C8 57.0 mm to (157.6, 78.3)
- moved G2 57.0 mm to (161.7, 70.7)
- moved Q13 57.0 mm to (215.3, 70.8)
- moved Q14 57.0 mm to (222.7, 70.7)
- moved Q15 57.0 mm to (229.7, 70.7)
- moved Q16 57.0 mm to (237.1, 70.9)
- moved R7 57.0 mm to (168.6, 76.4)
- moved C11 44.6 mm to (159.1, 127.6)
- moved G3 44.6 mm to (158.1, 123.2)
- moved Q17 44.6 mm to (170.6, 123.9)
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- renumbered C4 to C11, C5 to C12, C1 to C14, C2 to C15, C3 to C16, C10 to C6, C11 to C8, U3 to G2, U1 to G3, Q21 to Q13, Q22 to Q14, Q23 to Q15, Q24 to Q16, Q1 to Q17, Q2 to Q18, Q3 to Q19, Q4 to Q20, Q5 to Q21, Q6 to Q22, Q7 to Q23, Q8 to Q24, R2 to R10, R3 to R11, R4 to R12, R1 to R6, R9 to R7, R10 to R8, R8 to R9, SW1 to SW2, U13 to U2, U11 to U3, U10 to U4
Connections:
- net /CS renamed CS
- net /SCK renamed SCK
- net /SI renamed SI
- net /SO renamed SO
- A2 pad 27: Net-(A2-+5V) -> +5V
- C12 pad 2: Net-(D2-K) -> Net-(G3-VB)
- C13 pad 1: +5V -> GND
- C13 pad 2: GND -> Net-(J3-Pin_3)
- C7 pad 2: +12V -> C+
- C8 pad 2: Net-(D4-K) -> Net-(G2-VB)
- C9 pad 2: Net-(J7-Pin_1) -> C-
- D2 pad 1: Net-(D2-K) -> Net-(G2-VB)
- D3 pad 1: Net-(D3-K) -> Net-(G3-VB)
- G2 pad 8: Net-(D4-K) -> Net-(G2-VB)
- G3 pad 8: Net-(D2-K) -> Net-(G3-VB)
- J1 pad 2: /CAN HIGH -> /CAN LOW
- Q10 pad 1: Net-(J7-Pin_1) -> Net-(J3-Pin_2)
- Q10 pad 2: Net-(J7-Pin_1) -> Net-(J3-Pin_2)
- Q10 pad 3: Net-(J7-Pin_1) -> Net-(J3-Pin_2)
- Q10 pad 4: Net-(J7-Pin_1) -> Net-(J3-Pin_2)
- Q11 pad 1: Net-(J7-Pin_1) -> Net-(J3-Pin_2)
- Q11 pad 2: Net-(J7-Pin_1) -> Net-(J3-Pin_2)
- Q11 pad 3: Net-(J7-Pin_1) -> Net-(J3-Pin_2)
- Q11 pad 4: Net-(J7-Pin_1) -> Net-(J3-Pin_2)
- Q12 pad 1: Net-(J7-Pin_1) -> Net-(J3-Pin_2)
- Q12 pad 2: Net-(J7-Pin_1) -> Net-(J3-Pin_2)
- Q12 pad 3: Net-(J7-Pin_1) -> Net-(J3-Pin_2)
- Q12 pad 4: Net-(J7-Pin_1) -> Net-(J3-Pin_2)
- Q13 pad 5: Net-(J6-Pin_1) -> Net-(J3-Pin_2)
- Q13 pad 6: Net-(J6-Pin_1) -> Net-(J3-Pin_2)
- Q13 pad 7: Net-(J6-Pin_1) -> Net-(J3-Pin_2)
- Q13 pad 8: Net-(J6-Pin_1) -> Net-(J3-Pin_2)
- Q14 pad 5: Net-(J6-Pin_1) -> Net-(J3-Pin_2)
- Q14 pad 6: Net-(J6-Pin_1) -> Net-(J3-Pin_2)
- Q14 pad 7: Net-(J6-Pin_1) -> Net-(J3-Pin_2)
- Q14 pad 8: Net-(J6-Pin_1) -> Net-(J3-Pin_2)
- Q15 pad 5: Net-(J6-Pin_1) -> Net-(J3-Pin_2)
- Q15 pad 6: Net-(J6-Pin_1) -> Net-(J3-Pin_2)
- Q15 pad 7: Net-(J6-Pin_1) -> Net-(J3-Pin_2)
- Q15 pad 8: Net-(J6-Pin_1) -> Net-(J3-Pin_2)
- Q16 pad 5: Net-(J6-Pin_1) -> Net-(J3-Pin_2)
- Q16 pad 6: Net-(J6-Pin_1) -> Net-(J3-Pin_2)
- Q16 pad 7: Net-(J6-Pin_1) -> Net-(J3-Pin_2)
- Q16 pad 8: Net-(J6-Pin_1) -> Net-(J3-Pin_2)
- Q17 pad 1: Net-(J8-Pin_1) -> Net-(J3-Pin_3)
- Q17 pad 2: Net-(J8-Pin_1) -> Net-(J3-Pin_3)
- Q17 pad 3: Net-(J8-Pin_1) -> Net-(J3-Pin_3)
- Q17 pad 4: Net-(J8-Pin_1) -> Net-(J3-Pin_3)
- Q18 pad 1: Net-(J8-Pin_1) -> Net-(J3-Pin_3)
- Q18 pad 2: Net-(J8-Pin_1) -> Net-(J3-Pin_3)
- Q18 pad 3: Net-(J8-Pin_1) -> Net-(J3-Pin_3)
- Q18 pad 4: Net-(J8-Pin_1) -> Net-(J3-Pin_3)
- Q19 pad 1: Net-(J8-Pin_1) -> Net-(J3-Pin_3)
- Q19 pad 2: Net-(J8-Pin_1) -> Net-(J3-Pin_3)
- Q19 pad 3: Net-(J8-Pin_1) -> Net-(J3-Pin_3)
- Q19 pad 4: Net-(J8-Pin_1) -> Net-(J3-Pin_3)
- Q20 pad 1: Net-(J8-Pin_1) -> Net-(J3-Pin_3)
- Q20 pad 2: Net-(J8-Pin_1) -> Net-(J3-Pin_3)
- Q20 pad 3: Net-(J8-Pin_1) -> Net-(J3-Pin_3)
- Q20 pad 4: Net-(J8-Pin_1) -> Net-(J3-Pin_3)
- Q21 pad 5: Net-(J8-Pin_1) -> Net-(J3-Pin_3)
- Q21 pad 6: Net-(J8-Pin_1) -> Net-(J3-Pin_3)
- Q21 pad 7: Net-(J8-Pin_1) -> Net-(J3-Pin_3)
- Q21 pad 8: Net-(J8-Pin_1) -> Net-(J3-Pin_3)
- Q22 pad 5: Net-(J8-Pin_1) -> Net-(J3-Pin_3)
- Q22 pad 6: Net-(J8-Pin_1) -> Net-(J3-Pin_3)
- Q22 pad 7: Net-(J8-Pin_1) -> Net-(J3-Pin_3)
- Q22 pad 8: Net-(J8-Pin_1) -> Net-(J3-Pin_3)
- Q23 pad 5: Net-(J8-Pin_1) -> Net-(J3-Pin_3)
- Q23 pad 6: Net-(J8-Pin_1) -> Net-(J3-Pin_3)
- Q23 pad 7: Net-(J8-Pin_1) -> Net-(J3-Pin_3)
- Q23 pad 8: Net-(J8-Pin_1) -> Net-(J3-Pin_3)
- Q24 pad 5: Net-(J8-Pin_1) -> Net-(J3-Pin_3)
- Q24 pad 6: Net-(J8-Pin_1) -> Net-(J3-Pin_3)
- Q24 pad 7: Net-(J8-Pin_1) -> Net-(J3-Pin_3)
- Q24 pad 8: Net-(J8-Pin_1) -> Net-(J3-Pin_3)
- Q9 pad 1: Net-(J7-Pin_1) -> Net-(J3-Pin_2)
- Q9 pad 2: Net-(J7-Pin_1) -> Net-(J3-Pin_2)
- Q9 pad 3: Net-(J7-Pin_1) -> Net-(J3-Pin_2)
- Q9 pad 4: Net-(J7-Pin_1) -> Net-(J3-Pin_2)
- R11 pad 2: Net-(J8-Pin_1) -> Net-(J3-Pin_3)
- R7 pad 2: Net-(Q17-GATE) (its old number) -> Net-(Q10-GATE)
- R8 pad 2: Net-(J6-Pin_1) -> Net-(J3-Pin_2)
- U3 pad 1: Net-(U11-TXCAN) -> Net-(U1-TXD)
- U3 pad 2: Net-(U11-RXCAN) -> Net-(U1-RXD)
- U3 pad 7: unconnected-(U11-OSC2-Pad7) -> C+
- U3 pad 8: unconnected-(U11-OSC1-Pad8) -> C-
- U4 pad 1: Net-(D1-K) -> Net-(U4-VIN)
Routing:
- net Net-(Q17-GATE): track 66.6 -> 39.7 mm
- net Net-(Q21-GATE): track 72.2 -> 46.1 mm
- net Net-(G3-VB): track 0.00 -> 15.8 mm, vias 0 -> 2
- net Net-(D2-K): track 12.0 -> 0.00 mm, vias 2 -> 0
- net +12V: track 21.1 -> 30.3 mm
- net Net-(J8-Pin_1): track 6.15 -> 0.00 mm
- net Net-(G3-VS): track 6.75 -> 8.54 mm
- net Net-(G3-LO): track 45.4 -> 46.2 mm
- added copper zone on F.Cu, net GND
- added copper zone on F.Cu, net Net-(J3-Pin_3)
- removed copper zone on B.Cu, net GND
- removed copper zone on F.Cu, net Net-(J8-Pin_1)

Commit message: mosfet
Parts:
- moved R4 38.1 mm to (113.3, 73.7)
- moved R12 35.2 mm to (161.8, 131.4)
- moved D3 1.42 mm to (152.4, 115.6), turned to -90 degrees
Routing:
- net Net-(G3-LO): track 46.2 -> 10.9 mm
- net Net-(Q21-GATE): track 46.1 -> 81.2 mm
- net +12V: track 30.3 -> 20.1 mm
- net Net-(G3-VB): track 15.8 -> 20.4 mm
- net Net-(G3-HO): track 14.0 -> 15.4 mm
