File: _autosave-Urban MC.kicad_pcb (KiCad board)
At the start: 6 copper layers, 146.1 x 125.2 mm, 88 parts, among them J1 CAN, J2 UART_DYNO, J4 VBAT, J5 PWR_HALL, J6 HALL_SENSORS, J7 Conn_01x15_Socket, J8 Conn_02x03_CUSTOM, Q1 NTBLS0D8N08XTXG, Q2 NTBLS0D8N08XTXG, Q3 NTBLS0D8N08XTXG, Q4 NTBLS0D8N08XTXG, Q5 NTBLS0D8N08XTXG, Q6 NTBLS0D8N08XTXG, SW1 CAN_TERM, SW2 SW_MEC_5E, U1 MCP2561/2, U2 MCP4725, U3 MCP2515-xSO, Y1 8MHz

Commit message: 2026-2027 initial fixes from V1.2
Parts:
- removed the C14 at (228.5, 133.5)
Changed lines of the file:
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@@
 		)
-	)
-	(footprint "urban_mc_custom_footprints:CAPPRD750W80D1600H2500"
-		(layer "F.Cu")
-		(at 228.5 133.5 180)
-		(property "Reference" "C14"
-			(at 7.426 -6.7056 90)
-			(layer "F.SilkS")
-			(effects
-				(font
-					(size 1 1)
-					(thickness 0.15)
-				)
-			)
-		)
-		(property "Value" "1m"
-			(at -3.3436 -4.1656 90)
-			(layer "F.Fab")
-			(effects
-				(font
-					(size 1 1)
-					(thickness 0.15)
-				)
-			)
-		)
-		(property "Datasheet" "https://www.bourns.com/docs/Product-Datasheets/PTVS1-xxxC-H.pdf"
-			(at 0 0 0)
-			(layer "F.Fab")
-			(hide yes)
-			(effects
-				(font
-					(size 1.27 1.27)
-					(thickness 0.15)
-				)
-			)
-		)
-		(property "Description" "Polarized capacitor"
-			(at 0 0 0)
-			(layer "F.Fab")
-			(hide yes)
-			(effects
-				(font
-					(size 1.27 1.27)
-					(thickness 0.15)
-				)
-			)
-		)
-		(attr through_hole)
-		(fp_circle
-			(center 0 0)
-			(end 8 0)
-			(stroke
-				(width 0.127)
-				(type solid)
-			)
-			(fill no)
-			(layer "F.SilkS")
-		)
-		(fp_circle
-			(center -8.75 0)
-			(end -8.65 0)
-			(stroke
-				(width 0.2)
-				(type solid)
-			)
-			(fill no)
-			(layer "F.SilkS")
-		)
-		(fp_circle
-			(center 0 0)
-			(end 8.25 0)
-			(stroke
-				(width 0.05)
-				(type solid)
-			)
-			(fill no)
-			(layer "F.CrtYd")
-		)
-		(fp_circle
-			(center 0 0)
-			(end 8 0)
-			(stroke
-				(width 0.127)
-				(type solid)
-			)
-			(fill no)
-			(layer "F.Fab")
-		)
-		(fp_circle
-			(center -8.75 0)
-			(end -8.65 0)
-			(stroke
-				(width 0.2)
-				(type solid)
-			)
-			(fill no)
-			(layer "F.Fab")
-		)
-		(pad "1" thru_hole rect
-			(at -3.75 0 180)
-			(size 1.4 1.4)
-			(drill 1.05)
-			(layers "*.Cu" "*.Mask")
-			(remove_unused_layers no)
-			(pintype "passive")
-			(solder_mask_margin 0.102)
-		)
-		(pad "2" thru_hole circle
-			(at 3.75 0 180)
-			(size 1.4 1.4)
-			(drill 1.05)
-			(layers "*.Cu" "*.Mask")
-			(remove_unused_layers no)
-			(pintype "passive")
-			(solder_mask_margin 0.102)
-		)
-		(embedded_fonts no)
 	)
 	(footprint "Resistor_SMD:R_0805_2012Metric"
